Commit message: 调整相机高度和stack方向,以及修改说明文档

File: spark_v05/spark/spark_description/urdf/sensors/spark_camera.urdf (robot description, URDF)
Before this commit: robot camera_frame, 5 links, 5 joints
Joints:
- joint camera_link_joint: origin xyz=0.0936242 0 0.6279500 rpy=0 0 0 -> xyz=0.0936242 0 0.6629500 rpy=0 0 0

File: spark_v05/spark/spark_description/urdf/stack/spark_stack.urdf (robot description, URDF)
Before this commit: robot spark_stack, 1 links, 1 joints
Joints:
- joint spark_stack_joint: origin xyz=0 0 0 rpy=0 0 0 -> xyz=0 0 0 rpy=0 0 3.141592
