Commit message: 修改urdf文件模型比例

File: spark_v05/spark/spark_description/urdf/base/spark_base.urdf (robot description, URDF)
Before this commit: robot spark_base_link, 20 links, 19 joints
Links:
- link left_wheel_link: geometry collision mesh filename=package://spark_description/meshes/spark/base/left_wheel.DAE scale=0.001 0.001 0.001; visual mesh filename=package://spark_description/meshes/spark/base/left_wheel.DAE scale=0.001 0.001 0.001
- link right_wheel_link: geometry collision mesh filename=package://spark_description/meshes/spark/base/right_wheel.D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 scale=0.001 0.001 0.001; visual mesh filename=package://spark_description/meshes/spark/base/right_wheel.D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 scale=0.001 0.001 0.001
- link room_base_link: geometry collision mesh filename=package://spark_description/meshes/spark/base/spark_base.DAE scale=0.001 0.001 0.001; visual mesh filename=package://spark_description/meshes/spark/base/spark_base.DAE scale=0.001 0.001 0.001

File: spark_v05/spark/spark_description/urdf/sensors/spark_camera.urdf (robot description, URDF)
Before this commit: robot camera_frame, 5 links, 5 joints
Links:
- link camera_link: geometry collision mesh filename=package://spark_description/meshes/spark/sensors/spark_came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 scale=0.001 0.001 0.001; visual mesh filename=package://spark_description/meshes/spark/sensors/spark_came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 scale=0.001 0.001 0.001

File: spark_v05/spark/spark_description/urdf/stack/spark_stack.urdf (robot description, URDF)
Before this commit: robot spark_stack, 1 links, 1 joints
Links:
- link spark_stack: geometry collision mesh filename=package://spark_description/meshes/spark/stack/spark_stack.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 scale=0.001 0.001 0.001; visual mesh filename=package://spark_description/meshes/spark/stack/spark_stack.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 scale=0.001 0.001 0.001
