Commit message: 删除旧雷达，加入新雷达Delta-III驱动,此版本之后不再支持c0602银色版本的雷达。默认为Delta-III雷达。

File: src/spark/spark_description/urdf/sensors/spark_lidar.urdf (robot description, URDF)
Before this commit: robot lidar_frame, 1 links, 1 joints
Joints:
- joint lidar_joint: origin xyz=0 0 0.08 rpy=3.14 3.14 3.75 -> xyz=0 0 0.08 rpy=0 0 3.14
