Commit message: delete some unused files. add /imu_data topic to publish. bugfixes for the rtabmap when the ubuntu16.04 is upgraded to the newest version.

File: src/spark/spark_description/urdf/base/spark_base.urdf (robot description, URDF)
Before this commit: robot spark_base_link, 20 links, 19 joints
Links:
- added link IMU_link
Joints:
- added joint IMU_joint: type fixed, parent base_link, child IMU_link, origin xyz=0.104 -0.09 0.065 rpy=0 0 1.570796327
